Commit message: try to learn from untree

File: src/balance_description/urdf/balance.xacro (robot description, xacro)
@@ -2,6 +2,6 @@
 <robot xmlns:xacro="http://www.ros.org/wiki/xacro" name="diffdrive_robot">
     <xacro:include filename="$(find balance_description)/urdf/balance_description.xacro" />
-    <xacro:include filename="$(find balance_description)/urdf/balance_control.xacro" />
+    <!-- <xacro:include filename="$(find balance_description)/urdf/balance_control.xacro" /> -->
     <xacro:balance_robot />
-    <xacro:balance_ros2_control />
+    <!-- <xacro:balance_ros2_control /> -->
 </robot>

File: src/balance_description/urdf/balance_description.xacro (robot description, xacro)
@@ -2,8 +2,6 @@
 <robot xmlns:xacro="http://www.ros.org/wiki/xacro">
     <xacro:macro name="balance_robot" >
-        <xacro:property name="mesh_path" value="/home/emopointer/simulation_ws/src/balance_description/meshes"/>
-        <!-- gazebo -->
-        <!-- <xacro:property name="mesh_path" value="package://balance_description/meshes"/> -->
-        <!-- rviz -->
+        <xacro:property name="mesh_path" value="file://$(find balance_description)/meshes"/>
+        <!-- <xacro:property name="mesh_path" value="../meshes"/> -->
         <!-- macro -->
         <xacro:macro name="visual_and_collision" params="link_name mesh_file color xyz rpy">
@@ -102,6 +100,6 @@
                 effort="0"
                 velocity="0" />
-            <dynamics damping="0.5"/>
-            <initial_position>6.2</initial_position>
+            <dynamics damping="1"/>
+            <!-- <initial_position>6.2</initial_position> -->
         </joint>
         <joint
@@ -122,6 +120,6 @@
                 effort="0"
                 velocity="0" />
-            <dynamics damping="0.5"/>
-            <initial_position>0</initial_position>
+            <dynamics damping="1"/>
+            <!-- <initial_position>5.5</initial_position> -->
         </joint>
         <joint
@@ -142,6 +140,6 @@
                 effort="0"
                 velocity="0" />
-            <dynamics damping="0.5"/>
-            <initial_position>0</initial_position>
+            <dynamics damping="1"/>
+            <!-- <initial_position>0</initial_position> -->
         </joint>
         <joint
@@ -162,6 +160,6 @@
                 effort="0"
                 velocity="0" />
-            <dynamics damping="0.5"/>
-            <initial_position>6.2</initial_position>
+            <dynamics damping="1"/>
+            <!-- <initial_position>6.2</initial_position> -->
         </joint>
         <joint
@@ -182,6 +180,6 @@
                 effort="0"
                 velocity="0" />
-            <dynamics damping="0.5"/>
-            <initial_position>0</initial_position>
+            <dynamics damping="1"/>
+            <!-- <initial_position>0</initial_position> -->
         </joint>
         <joint
@@ -202,6 +200,6 @@
                 effort="0"
                 velocity="0" />
-            <dynamics damping="0.5"/>
-            <initial_position>0</initial_position>
+            <dynamics damping="1"/>
+            <!-- <initial_position>0</initial_position> -->
         </joint>
     </xacro:macro>

Commit message: import gazebo normally

File: src/balance_description/urdf/balance.xacro (robot description, xacro)
@@ -2,6 +2,6 @@
 <robot xmlns:xacro="http://www.ros.org/wiki/xacro" name="diffdrive_robot">
     <xacro:include filename="$(find balance_description)/urdf/balance_description.xacro" />
-    <!-- <xacro:include filename="$(find balance_description)/urdf/balance_control.xacro" /> -->
+    <xacro:include filename="$(find balance_description)/urdf/balance_control.xacro" />
     <xacro:balance_robot />
-    <!-- <xacro:balance_ros2_control /> -->
+    <xacro:balance_ros2_control />
 </robot>

File: src/balance_description/urdf/balance_control.xacro (robot description, xacro)
@@ -8,4 +8,78 @@
             <plugin>gazebo_ros2_control/GazeboSystem</plugin>
             </hardware>
+            <!-- <gazebo>
+                <plugin name="3dplot" filename="libLinkPlot3DPlugin.so">
+                    <frequency>10</frequency>
+                    <plot>
+                        <link>base_link</link>
+                        <pose>0 0 0 0 0 0</pose>
+                        <material>Gazebo/Yellow</material>
+                    </plot>
+                </plugin>
+            </gazebo> -->
+            <!-- <gazebo reference="imu_link">
+                <gravity>true</gravity>
+                <sensor name="imu_sensor" type="imu">
+                    <always_on>true</always_on>
+                    <update_rate>1000</update_rate>
+                    <visualize>true</visualize>
+                    <topic>__default_topic__</topic>
+                    <plugin filename="libgazebo_ros_imu_sensor.so" name="imu_plugin">
+                        <topicName>trunk_imu</topicName>
+                        <bodyName>imu_link</bodyName>
+                        <updateRateHZ>1000.0</updateRateHZ>
+                        <gaussianNoise>0.0</gaussianNoise>
+                        <xyzOffset>0 0 0</xyzOffset>
+                        <rpyOffset>0 0 0</rpyOffset>
+                        <frameName>imu_link</frameName>
+                    </plugin>
+                    <pose>0 0 0 0 0 0</pose>
+                </sensor>
+            </gazebo> -->
+            <gazebo>
+                <plugin filename="libgazebo_ros2_control.so" name="gazebo_ros2_control">
+                <parameters>$(find balance_description)/config/controller.yaml</parameters>
+                </plugin>
+            </gazebo>
+            <gazebo reference="base_link">
+                <material>Gazebo/Green</material>
+                <turnGravityOff>false</turnGravityOff>
+            </gazebo>
+            <gazebo reference="thigh1_Link">
+                <mu1>0.2</mu1>
+                <mu2>0.2</mu2>
+                <kp  value="1000000.0"/>
+                <kd  value="1.0"/>
+            </gazebo>
+            <gazebo reference="calf1_Link">
+                <mu1>0.2</mu1>
+                <mu2>0.2</mu2>
+                <kp  value="1000000.0"/>
+                <kd  value="1.0"/>
+            </gazebo>
+            <gazebo reference="wheel1_Link">
+                <mu1>0.2</mu1>
+                <mu2>0.2</mu2>
+                <kp  value="1000000.0"/>
+                <kd  value="1.0"/>
+            </gazebo>
+            <gazebo reference="thigh2_Link">
+                <mu1>0.2</mu1>
+                <mu2>0.2</mu2>
+                <kp  value="1000000.0"/>
+                <kd  value="1.0"/>
+            </gazebo>
+            <gazebo reference="calf2_Link">
+                <mu1>0.2</mu1>
+                <mu2>0.2</mu2>
+                <kp  value="1000000.0"/>
+                <kd  value="1.0"/>
+            </gazebo>
+            <gazebo reference="wheel2_Link">
+                <mu1>0.2</mu1>
+                <mu2>0.2</mu2>
+                <kp  value="1000000.0"/>
+                <kd  value="1.0"/>
+            </gazebo>
             <joint name="joint1">
                 <command_interface name="position"/>
@@ -13,5 +87,5 @@
                 <state_interface name="position"/>
                 <!-- <state_interface name="effort"/> -->
-                <param name="initial_position">6.2</param>
+                <param name="initial_position">0.0</param>
             </joint>
             <joint name="joint2">
@@ -36,5 +110,5 @@
                 <state_interface name="position"/>
                 <!-- <state_interface name="effort"/> -->
-                <param name="initial_position">6.2</param>
+                <param name="initial_position">0.0</param>
             </joint>
             <joint name="joint5">
@@ -55,10 +129,4 @@
             </joint>
         </ros2_control>
-            <!-- Gazebo 插件 -->
-        <gazebo>
-            <plugin filename="libgazebo_ros2_control.so" name="gazebo_ros2_control">
-            <parameters>$(find balance_description)/config/controller.yaml</parameters>
-            </plugin>
-        </gazebo>
     </xacro:macro>
 </robot>

File: src/balance_description/urdf/balance_description.xacro (robot description, xacro)
@@ -82,4 +82,13 @@
             <xacro:visual_and_collision link_name="wheel2_Link" mesh_file="wheel2_Link.STL" color="red" xyz="0 0 0" rpy="0 0 0"/>
         </link>
+        <!-- <link name="imu_link">
+            <inertial>
+            <origin xyz="-0.00112 0.03727 -0.00505" rpy="0 0 0"/>
+            <mass value="2.2956"/>
+            <inertia ixx="0.003765" ixy="-8.39e-6" ixz="1.11e-7" iyy="0.009989" iyz="-7.96e-8" izz="0.008215"/>
+            </inertial>
+            <xacro:visual_and_collision link_name="base_link" mesh_file="base_link.STL" color="silver"
+                xyz="0 0 0" rpy="1.57 0 3.14"/>
+        </link> -->
         <!-- joints -->
         <joint
@@ -96,10 +105,10 @@
                 xyz="0 0 1" />
             <limit
-                lower="5.9"
-                upper="7.39"
-                effort="0"
-                velocity="0" />
-            <dynamics damping="1"/>
-            <!-- <initial_position>6.2</initial_position> -->
+                lower="-0.38"
+                upper="1.11"
+                effort="23"
+                velocity="30" />
+            <dynamics damping="1"/>
+            <initial_position>0.0</initial_position>
         </joint>
         <joint
@@ -116,10 +125,10 @@
                 xyz="0 0 -1" />
             <limit
-                lower="5"
-                upper="6.74"
-                effort="0"
-                velocity="0" />
-            <dynamics damping="1"/>
-            <!-- <initial_position>5.5</initial_position> -->
+                lower="-1.28"
+                upper="0.46"
+                effort="23"
+                velocity="30" />
+            <dynamics damping="1"/>
+            <initial_position>0.0</initial_position>
         </joint>
         <joint
@@ -136,10 +145,8 @@
                 xyz="0 0 -1" />
             <limit
-                lower="0"
-                upper="0"
-                effort="0"
-                velocity="0" />
-            <dynamics damping="1"/>
-            <!-- <initial_position>0</initial_position> -->
+                effort="27"
+                velocity="30" />
+            <dynamics damping="1"/>
+            <initial_position>0.0</initial_position>
         </joint>
         <joint
@@ -156,10 +163,10 @@
                 xyz="0 0 1" />
             <limit
-                lower="5.45"
-                upper="6.95"
-                effort="0"
-                velocity="0" />
-            <dynamics damping="1"/>
-            <!-- <initial_position>6.2</initial_position> -->
+                lower="-0.83"
+                upper="0.67"
+                effort="27"
+                velocity="30" />
+            <dynamics damping="1"/>
+            <initial_position>0.0</initial_position>
         </joint>
         <joint
@@ -178,8 +185,8 @@
                 lower="-0.68"
                 upper="1.06"
-                effort="0"
-                velocity="0" />
-            <dynamics damping="1"/>
-            <!-- <initial_position>0</initial_position> -->
+                effort="27"
+                velocity="30" />
+            <dynamics damping="1"/>
+            <initial_position>0.0</initial_position>
         </joint>
         <joint
@@ -196,10 +203,8 @@
                 xyz="0 0 1" />
             <limit
-                lower="0"
-                upper="0"
-                effort="0"
-                velocity="0" />
-            <dynamics damping="1"/>
-            <!-- <initial_position>0</initial_position> -->
+                effort="27"
+                velocity="30" />
+            <dynamics damping="1"/>
+            <initial_position>0.0</initial_position>
         </joint>
     </xacro:macro>
