Commit message: gazebo hardware interface is ok

File: src/balance_description/urdf/balance_control.xacro (robot description, xacro)
@@ -5,5 +5,6 @@
         <ros2_control name="balance_control" type="system">
             <hardware>
-            <plugin>balance_hardware_interface/BalanceHardwareInterface</plugin>
+            <!-- <plugin>balance_hardware_interface/BalanceHardwareInterface</plugin> -->
+            <plugin>gazebo_ros2_control/GazeboSystem</plugin>
             </hardware>
             <joint name="joint1">
@@ -12,5 +13,5 @@
                 <state_interface name="position"/>
                 <!-- <state_interface name="effort"/> -->
-                <param name="initial_position">0.0</param>
+                <param name="initial_position">6.2</param>
             </joint>
             <joint name="joint2">
@@ -35,5 +36,5 @@
                 <state_interface name="position"/>
                 <!-- <state_interface name="effort"/> -->
-                <param name="initial_position">0.0</param>
+                <param name="initial_position">6.2</param>
             </joint>
             <joint name="joint5">
@@ -55,9 +56,9 @@
         </ros2_control>
             <!-- Gazebo 插件 -->
-        <!-- <gazebo>
+        <gazebo>
             <plugin filename="libgazebo_ros2_control.so" name="gazebo_ros2_control">
             <parameters>$(find balance_description)/config/controller.yaml</parameters>
             </plugin>
-        </gazebo> -->
+        </gazebo>
     </xacro:macro>
 </robot>

File: src/balance_description/urdf/balance_description.xacro (robot description, xacro)
@@ -2,11 +2,12 @@
 <robot xmlns:xacro="http://www.ros.org/wiki/xacro">
     <xacro:macro name="balance_robot" >
-        <!-- <xacro:property name="mesh_path" value="/home/emopointer/simulation_ws/src/balance_description/meshes"/> -->
+        <xacro:property name="mesh_path" value="/home/emopointer/simulation_ws/src/balance_description/meshes"/>
         <!-- gazebo -->
-        <xacro:property name="mesh_path" value="package://balance_description/meshes"/>
+        <!-- <xacro:property name="mesh_path" value="package://balance_description/meshes"/> -->
         <!-- rviz -->
         <!-- macro -->
-        <xacro:macro name="visual_and_collision" params="link_name mesh_file color">
+        <xacro:macro name="visual_and_collision" params="link_name mesh_file color xyz rpy">
             <visual>
+            <origin xyz="${xyz}" rpy="${rpy}"/>
             <geometry>
                 <mesh filename="${mesh_path}/${mesh_file}"/>
@@ -17,4 +18,5 @@
             </visual>
             <collision>
+            <origin xyz="${xyz}" rpy="${rpy}"/>
             <geometry>
                 <mesh filename="${mesh_path}/${mesh_file}"/>
@@ -31,5 +33,6 @@
             <!-- mass martrix -->
             </inertial>
-            <xacro:visual_and_collision link_name="base_link" mesh_file="base_link.STL" color="silver"/>
+            <xacro:visual_and_collision link_name="base_link" mesh_file="base_link.STL" color="silver"
+                xyz="0 0 0" rpy="1.57 0 3.14"/>
         </link>
         <link name="thigh1_Link">
@@ -39,5 +42,5 @@
             <inertia ixx="0.000242" ixy="0.000152" ixz="0" iyy="0.000196" iyz="0" izz="0.000432"/>
             </inertial>
-            <xacro:visual_and_collision link_name="thigh1_Link" mesh_file="thigh1_Link.STL" color="blue"/>
+            <xacro:visual_and_collision link_name="thigh1_Link" mesh_file="thigh1_Link.STL" color="blue" xyz="0 0 0" rpy="0 0 0"/>
         </link>
         <link name="calf1_Link">
@@ -47,5 +50,5 @@
             <inertia ixx="0.000443" ixy="-0.000512" ixz="0" iyy="0.000859" iyz="0" izz="0.001298"/>
             </inertial>
-            <xacro:visual_and_collision link_name="calf1_Link" mesh_file="calf1_Link.STL" color="silver"/>
+            <xacro:visual_and_collision link_name="calf1_Link" mesh_file="calf1_Link.STL" color="silver" xyz="0 0 0" rpy="0 0 0"/>
         </link>
         <link name="wheel1_Link">
@@ -55,5 +58,5 @@
             <inertia ixx="0.00354" ixy="0" ixz="0" iyy="0.00354" iyz="0" izz="0.00682"/>
             </inertial>
-            <xacro:visual_and_collision link_name="wheel1_Link" mesh_file="wheel1_Link.STL" color="red"/>
+            <xacro:visual_and_collision link_name="wheel1_Link" mesh_file="wheel1_Link.STL" color="red" xyz="0 0 0" rpy="0 0 0"/>
         </link>
         <link name="thigh2_Link">
@@ -63,5 +66,5 @@
             <inertia ixx="0.000114" ixy="0.000112" ixz="0" iyy="0.000324" iyz="0" izz="0.000432"/>
             </inertial>
-            <xacro:visual_and_collision link_name="thigh2_Link" mesh_file="thigh2_Link.STL" color="blue"/>
+            <xacro:visual_and_collision link_name="thigh2_Link" mesh_file="thigh2_Link.STL" color="blue" xyz="0 0 0" rpy="0 0 0"/>
         </link>
         <link name="calf2_Link">
@@ -71,5 +74,5 @@
             <inertia ixx="0.000596" ixy="0.000549" ixz="0" iyy="0.000706" iyz="0" izz="0.001298"/>
             </inertial>
-            <xacro:visual_and_collision link_name="calf2_Link" mesh_file="calf2_Link.STL" color="silver"/>
+            <xacro:visual_and_collision link_name="calf2_Link" mesh_file="calf2_Link.STL" color="silver" xyz="0 0 0" rpy="0 0 0"/>
         </link>
         <link name="wheel2_Link">
@@ -79,52 +82,126 @@
             <inertia ixx="0.00354" ixy="0" ixz="0" iyy="0.00354" iyz="0" izz="0.00682"/>
             </inertial>
-            <xacro:visual_and_collision link_name="wheel2_Link" mesh_file="wheel2_Link.STL" color="red"/>
+            <xacro:visual_and_collision link_name="wheel2_Link" mesh_file="wheel2_Link.STL" color="red" xyz="0 0 0" rpy="0 0 0"/>
         </link>
         <!-- joints -->
-        <joint name="joint1" type="revolute">
-            <origin xyz="0.055 0.060 -0.179" rpy="0 0 0"/>
-            <parent link="base_link"/>
-            <child link="thigh1_Link"/>
-            <axis xyz="0 0 1"/>
-            <dynamics damping="0.5"/>
-            <limit lower="4.45" upper="7.39" effort="10" velocity="10"/>
-        </joint>
-        <joint name="joint2" type="revolute">
-            <origin xyz="0.0984 -0.1132 -0.0508" rpy="-3.1416 0 1.5708"/>
-            <parent link="thigh1_Link"/>
-            <child link="calf1_Link"/>
-            <axis xyz="0 0 -1"/>
-            <dynamics damping="0.5"/>
-            <limit lower="5" upper="8.96" effort="10" velocity="10"/>
-        </joint>
-        <joint name="joint3" type="continuous">
-            <origin xyz="-0.1992 -0.1338 0.0502" rpy="3.1416 0 1.5708"/>
-            <parent link="calf1_Link"/>
-            <child link="wheel1_Link"/>
-            <axis xyz="0 0 -1"/>
-            <dynamics damping="0.5"/>
-        </joint>
-        <joint name="joint4" type="revolute">
-            <origin xyz="0.055 0.060 0.179" rpy="0 0 0"/>
-            <parent link="base_link"/>
-            <child link="thigh2_Link"/>
-            <axis xyz="0 0 1"/>
-            <dynamics damping="0.5"/>
-            <limit lower="3.81" upper="7.17" effort="10" velocity="10"/>
-        </joint>
-        <joint name="joint5" type="revolute">
-            <origin xyz="0.1373 -0.0604 0.0523" rpy="0 0 1.5708"/>
-            <parent link="thigh2_Link"/>
-            <child link="calf2_Link"/>
-            <axis xyz="0 0 -1"/>
-            <dynamics damping="0.5"/>
-            <limit lower="-3.36" upper="0.63" effort="10" velocity="10"/>
-        </joint>
-        <joint name="joint6" type="continuous">
-            <origin xyz="-0.1778 0.1612 0.0502" rpy="3.1416 0 1.5708"/>
-            <parent link="calf2_Link"/>
-            <child link="wheel2_Link"/>
-            <axis xyz="0 0 -1"/>
-            <dynamics damping="0.5"/>
+        <joint
+            name="joint1"
+            type="revolute">
+            <origin
+                xyz="-0.054991 -0.179 0.060002"
+                rpy="1.57 0 3.14" />
+            <parent
+                link="base_link" />
+            <child
+                link="thigh1_Link" />
+            <axis
+                xyz="0 0 1" />
+            <limit
+                lower="5.9"
+                upper="7.39"
+                effort="0"
+                velocity="0" />
+            <dynamics damping="0.5"/>
+            <initial_position>6.2</initial_position>
+        </joint>
+        <joint
+            name="joint2"
+            type="revolute">
+            <origin
+                xyz="0.098406 -0.11321 -0.0508"
+                rpy="-3.1416 0 1.5708" />
+            <parent
+                link="thigh1_Link" />
+            <child
+                link="calf1_Link" />
+            <axis
+                xyz="0 0 -1" />
+            <limit
+                lower="5"
+                upper="6.74"
+                effort="0"
+                velocity="0" />
+            <dynamics damping="0.5"/>
+            <initial_position>0</initial_position>
+        </joint>
+        <joint
+            name="joint3"
+            type="continuous">
+            <origin
+                xyz="-0.19921 -0.13384 0.0502"
+                rpy="3.1416 0 1.5708" />
+            <parent
+                link="calf1_Link" />
+            <child
+                link="wheel1_Link" />
+            <axis
+                xyz="0 0 -1" />
+            <limit
+                lower="0"
+                upper="0"
+                effort="0"
+                velocity="0" />
+            <dynamics damping="0.5"/>
+            <initial_position>0</initial_position>
+        </joint>
+        <joint
+            name="joint4"
+            type="revolute">
+            <origin
+                xyz="-0.054991 0.179 0.060002"
+                rpy="1.57 0 3.14" />
+            <parent
+                link="base_link" />
+            <child
+                link="thigh2_Link" />
+            <axis
+                xyz="0 0 1" />
+            <limit
+                lower="5.45"
+                upper="6.95"
+                effort="0"
+                velocity="0" />
+            <dynamics damping="0.5"/>
+            <initial_position>6.2</initial_position>
+        </joint>
+        <joint
+            name="joint5"
+            type="revolute">
+            <origin
+                xyz="0.13731 -0.06037 0.0523"
+                rpy="0 0 1.5708" />
+            <parent
+                link="thigh2_Link" />
+            <child
+                link="calf2_Link" />
+            <axis
+                xyz="0 0 1" />
+            <limit
+                lower="-0.68"
+                upper="1.06"
+                effort="0"
+                velocity="0" />
+            <dynamics damping="0.5"/>
+            <initial_position>0</initial_position>
+        </joint>
+        <joint
+            name="joint6"
+            type="continuous">
+            <origin
+                xyz="-0.177825913114533 0.161176749639925 0.0502000000001869"
+                rpy="3.14159265358979 0 1.5707963267949" />
+            <parent
+                link="calf2_Link" />
+            <child
+                link="wheel2_Link" />
+            <axis
+                xyz="0 0 1" />
+            <limit
+                lower="0"
+                upper="0"
+                effort="0"
+                velocity="0" />
+            <dynamics damping="0.5"/>
+            <initial_position>0</initial_position>
         </joint>
     </xacro:macro>

Commit message: position control is ok,but fly in gazebo

File: src/balance_description/urdf/balance_control.xacro (robot description, xacro)
@@ -37,49 +37,4 @@
                 </sensor>
             </gazebo> -->
-            <gazebo>
-                <plugin filename="libgazebo_ros2_control.so" name="gazebo_ros2_control">
-                <parameters>$(find balance_description)/config/controller.yaml</parameters>
-                </plugin>
-            </gazebo>
-            <gazebo reference="base_link">
-                <material>Gazebo/Green</material>
-                <turnGravityOff>false</turnGravityOff>
-            </gazebo>
-            <gazebo reference="thigh1_Link">
-                <mu1>0.2</mu1>
-                <mu2>0.2</mu2>
-                <kp  value="1000000.0"/>
-                <kd  value="1.0"/>
-            </gazebo>
-            <gazebo reference="calf1_Link">
-                <mu1>0.2</mu1>
-                <mu2>0.2</mu2>
-                <kp  value="1000000.0"/>
-                <kd  value="1.0"/>
-            </gazebo>
-            <gazebo reference="wheel1_Link">
-                <mu1>0.2</mu1>
-                <mu2>0.2</mu2>
-                <kp  value="1000000.0"/>
-                <kd  value="1.0"/>
-            </gazebo>
-            <gazebo reference="thigh2_Link">
-                <mu1>0.2</mu1>
-                <mu2>0.2</mu2>
-                <kp  value="1000000.0"/>
-                <kd  value="1.0"/>
-            </gazebo>
-            <gazebo reference="calf2_Link">
-                <mu1>0.2</mu1>
-                <mu2>0.2</mu2>
-                <kp  value="1000000.0"/>
-                <kd  value="1.0"/>
-            </gazebo>
-            <gazebo reference="wheel2_Link">
-                <mu1>0.2</mu1>
-                <mu2>0.2</mu2>
-                <kp  value="1000000.0"/>
-                <kd  value="1.0"/>
-            </gazebo>
             <joint name="joint1">
                 <command_interface name="position"/>
@@ -88,4 +43,6 @@
                 <!-- <state_interface name="effort"/> -->
                 <param name="initial_position">0.0</param>
+                <param name="min">-0.38</param>
+                <param name="max">1.11</param>
             </joint>
             <joint name="joint2">
@@ -95,4 +52,6 @@
                 <!-- <state_interface name="effort"/> -->
                 <param name="initial_position">0.0</param>
+                <param name="min">-1.28</param>
+                <param name="max">0..46</param>
             </joint>
             <joint name="joint3">
@@ -110,5 +69,7 @@
                 <state_interface name="position"/>
                 <!-- <state_interface name="effort"/> -->
-                <param name="initial_position">0.0</param>
+                <!-- <param name="initial_position">0.0</param> -->
+                <param name="min">-0.83</param>
+                <param name="max">0.67</param>
             </joint>
             <joint name="joint5">
@@ -118,4 +79,6 @@
                 <!-- <state_interface name="effort"/> -->
                 <param name="initial_position">0.0</param>
+                <param name="min">-0.68</param>
+                <param name="max">1.06</param>
             </joint>
             <joint name="joint6">
@@ -127,6 +90,59 @@
                 <!-- <state_interface name="effort"/> -->
                 <param name="initial_position">0.0</param>
+                <param name="min">-1</param>
+                <param name="max">1</param>
             </joint>
         </ros2_control>
+        <gazebo>
+            <plugin filename="libgazebo_ros2_control.so" name="gazebo_ros2_control">
+                <parameters>$(find balance_description)/config/controller.yaml</parameters>
+            </plugin>
+        </gazebo>
+            <gazebo reference="base_link">
+                <!-- <material>Gazebo/Green</material> -->
+                <turnGravityOff>true</turnGravityOff>
+            </gazebo>
+            <gazebo reference="thigh1_Link">
+                <mu1>0.2</mu1>
+                <mu2>0.2</mu2>
+                <kp  value="100000.0"/>
+                <kd  value="1000.0"/>
+                <turnGravityOff>true</turnGravityOff>
+            </gazebo>
+            <gazebo reference="calf1_Link">
+                <mu1>0.2</mu1>
+                <mu2>0.2</mu2>
+                <kp  value="100000.0"/>
+                <kd  value="1000.0"/>
+                <turnGravityOff>true</turnGravityOff>
+            </gazebo>
+            <gazebo reference="wheel1_Link">
+                <mu1>0.2</mu1>
+                <mu2>0.2</mu2>
+                <kp  value="100000.0"/>
+                <kd  value="1000.0"/>
+                <turnGravityOff>true</turnGravityOff>
+            </gazebo>
+            <gazebo reference="thigh2_Link">
+                <mu1>0.2</mu1>
+                <mu2>0.2</mu2>
+                <kp  value="100000.0"/>
+                <kd  value="1000.0"/>
+                <turnGravityOff>true</turnGravityOff>
+            </gazebo>
+            <gazebo reference="calf2_Link">
+                <mu1>0.2</mu1>
+                <mu2>0.2</mu2>
+                <kp  value="100000.0"/>
+                <kd  value="1000.0"/>
+                <turnGravityOff>true</turnGravityOff>
+            </gazebo>
+            <gazebo reference="wheel2_Link">
+                <mu1>0.2</mu1>
+                <mu2>0.2</mu2>
+                <kp  value="100000.0"/>
+                <kd  value="1000.0"/>
+                <turnGravityOff>true</turnGravityOff>
+            </gazebo>
     </xacro:macro>
 </robot>

File: src/balance_description/urdf/balance_description.xacro (robot description, xacro)
@@ -107,5 +107,5 @@
                 lower="-0.38"
                 upper="1.11"
-                effort="23"
+                effort="1"
                 velocity="30" />
             <dynamics damping="1"/>
@@ -127,6 +127,6 @@
                 lower="-1.28"
                 upper="0.46"
-                effort="23"
-                velocity="30" />
+                effort="1"
+                velocity="1" />
             <dynamics damping="1"/>
             <initial_position>0.0</initial_position>
@@ -145,6 +145,6 @@
                 xyz="0 0 -1" />
             <limit
-                effort="27"
-                velocity="30" />
+                effort="1"
+                velocity="1" />
             <dynamics damping="1"/>
             <initial_position>0.0</initial_position>
@@ -165,6 +165,6 @@
                 lower="-0.83"
                 upper="0.67"
-                effort="27"
-                velocity="30" />
+                effort="1"
+                velocity="1" />
             <dynamics damping="1"/>
             <initial_position>0.0</initial_position>
@@ -185,6 +185,6 @@
                 lower="-0.68"
                 upper="1.06"
-                effort="27"
-                velocity="30" />
+                effort="1"
+                velocity="1" />
             <dynamics damping="1"/>
             <initial_position>0.0</initial_position>
@@ -203,6 +203,6 @@
                 xyz="0 0 1" />
             <limit
-                effort="27"
-                velocity="30" />
+                effort="1"
+                velocity="1" />
             <dynamics damping="1"/>
             <initial_position>0.0</initial_position>
